File: HW/RenjiSystem.kicad_pcb (KiCad board)
At the start: 2 copper layers, 205.7 x 116.8 mm, 53 parts, among them J1 Screw_Terminal_AC100VHOT, J10 Conn_AE_LXDC55_5V, J11 Conn_AE_QFP100PR5_DIP_1_25, J12 Conn_AE_QFP100PR5_DIP_26_50, J13 Conn_AE_QFP100PR5_DIP_51_75, J14 Conn_AE_QFP100PR5_DIP_76_100, J15 Conn_LCD, J16 Conn_Ethernet, J17 Conn_UART1, J18 Conn_UART2, J19 Conn_Debug, J2 Screw_Terminal_AC100VCOLD, J20 Conn_SwitchBoard, J21 Conn_LEDIndicator, J22 Conn_Thermistor, J3 Screw_Terminal_UV_HOT, J4 Screw_Terminal_UV_COLD, J5 Screw_Terminal_HEATER_HOT, J6 Screw_Terminal_HEATER_COLD, J7 Screw_Terminal_FAN_HOT, J8 Screw_Terminal_FAN_COLD, J9 Conn_AE_LXDC55_3.3V, K1 G5Q-14_DC5, K2 G5Q-14_DC5, K3 G5Q-14_DC5, Q1 2SC1815, Q2 2SC1815, Q3 2SC1815, T1 Transformer_FS24-100-C2

Commit message: シルクで1ピンマーク追記
Other:
- board text added: "AC100V IN"
- board text added: "G"
- board text added: "I"
- board text added: "Instrument0"
- board text added: "Instrument1"
- board text added: "Instrument2"
- board text added: "O"
Changed lines of the file:
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@@
   (general
     (thickness 1.6)
-    (drawings 23)
+    (drawings 54)
     (tracks 357)
     (zones 0)
@@
     )
   )
+  (gr_text O (at 139.7 95.25) (layer F.SilkS)
+    (effects (font (size 1.5 1.5) (thickness 0.3)))
+  )
+  (gr_text I (at 134.62 95.25) (layer F.SilkS)
+    (effects (font (size 1.5 1.5) (thickness 0.3)))
+  )
+  (gr_text "G\n" (at 137.16 95.25) (layer F.SilkS)
+    (effects (font (size 1.5 1.5) (thickness 0.3)))
+  )
+  (gr_text O (at 139.7 125.73) (layer F.SilkS)
+    (effects (font (size 1.5 1.5) (thickness 0.3)))
+  )
+  (gr_text "G\n" (at 137.16 125.73) (layer F.SilkS)
+    (effects (font (size 1.5 1.5) (thickness 0.3)))
+  )
+  (gr_text I (at 134.62 125.73) (layer F.SilkS)
+    (effects (font (size 1.5 1.5) (thickness 0.3)))
+  )
+  (gr_circle (center 229.87 60.96) (end 230.12 60.96) (layer F.SilkS) (width 0.5))
+  (gr_circle (center 241.3 39.37) (end 241.55 39.37) (layer F.SilkS) (width 0.5))
+  (gr_circle (center 219.71 39.37) (end 219.96 39.37) (layer F.SilkS) (width 0.5))
+  (gr_circle (center 196.85 40.64) (end 197.1 40.64) (layer F.SilkS) (width 0.5))
+  (gr_circle (center 157.48 38.1) (end 157.73 38.1) (layer F.SilkS) (width 0.5))
+  (gr_text Instrument2 (at 135.89 27.94) (layer F.SilkS)
+    (effects (font (size 1.5 1.5) (thickness 0.3)))
+  )
+  (gr_text Instrument1 (at 104.14 27.94) (layer F.SilkS)
+    (effects (font (size 1.5 1.5) (thickness 0.3)))
+  )
+  (gr_text Instrument0 (at 71.12 27.94) (layer F.SilkS)
+    (effects (font (size 1.5 1.5) (thickness 0.3)))
+  )
+  (gr_line (start 152.4 26.67) (end 120.65 26.67) (layer F.SilkS) (width 0.2))
+  (gr_line (start 152.4 48.26) (end 152.4 26.67) (layer F.SilkS) (width 0.2))
+  (gr_line (start 120.65 48.26) (end 152.4 48.26) (layer F.SilkS) (width 0.2))
+  (gr_line (start 120.65 26.67) (end 120.65 48.26) (layer F.SilkS) (width 0.2))
+  (gr_line (start 119.38 48.26) (end 87.63 48.26) (layer F.SilkS) (width 0.2))
+  (gr_line (start 119.38 26.67) (end 119.38 48.26) (layer F.SilkS) (width 0.2))
+  (gr_line (start 87.63 26.67) (end 119.38 26.67) (layer F.SilkS) (width 0.2))
+  (gr_line (start 87.63 48.26) (end 87.63 26.67) (layer F.SilkS) (width 0.2))
+  (gr_line (start 86.36 26.67) (end 54.61 26.67) (layer F.SilkS) (width 0.2))
+  (gr_line (start 86.36 48.26) (end 86.36 26.67) (layer F.SilkS) (width 0.2))
+  (gr_line (start 54.61 48.26) (end 86.36 48.26) (layer F.SilkS) (width 0.2))
+  (gr_line (start 54.61 26.67) (end 54.61 48.26) (layer F.SilkS) (width 0.2))
+  (gr_text "AC100V IN" (at 41.91 110.49 90) (layer F.SilkS)
+    (effects (font (size 1.5 1.5) (thickness 0.3)))
+  )
+  (gr_line (start 39.37 128.27) (end 39.37 93.98) (layer F.SilkS) (width 0.2))
+  (gr_line (start 63.5 128.27) (end 39.37 128.27) (layer F.SilkS) (width 0.2))
+  (gr_line (start 63.5 93.98) (end 63.5 128.27) (layer F.SilkS) (width 0.2))
+  (gr_line (start 39.37 93.98) (end 63.5 93.98) (layer F.SilkS) (width 0.2))
   (gr_text "LAN8720A board" (at 176.53 67.31) (layer F.SilkS)
     (effects (font (size 1.5 1.5) (thickness 0.3)))
