File: HW/file5FF7CD1C.sch (KiCad schematic (older format))
At the start: 8 parts, among them J11 Conn_AE_QFP100PR5_DIP_1_25, J12 Conn_AE_QFP100PR5_DIP_26_50, J13 Conn_AE_QFP100PR5_DIP_51_75, J14 Conn_AE_QFP100PR5_DIP_76_100

Commit message: Ethernetボードの配置のためにレイアウト変更
Connections:
- net LED_SIGNAL0: now also J14.2 (Pin_2); no longer J13.4 (Pin_4)
- net LED_SIGNAL1: now also J14.3 (Pin_3); no longer J13.3 (Pin_3)
- net LED_SIGNAL2: now also J14.4 (Pin_4); no longer J13.5 (Pin_5)
- net LED_SIGNAL3: now also J14.5 (Pin_5); no longer J13.6 (Pin_6)
Changed lines of the file:
@@
 NoConn ~ 6000 3500
 NoConn ~ 6000 3400
-NoConn ~ 6000 3300
-NoConn ~ 6000 3200
-NoConn ~ 6500 3200
-NoConn ~ 6500 3100
 NoConn ~ 6500 3300
 NoConn ~ 6500 3400
@@
 Wire Bus Line
 	9950 2550 10200 2550
-Text Label 5150 1450 0    50   ~ 0
+Text Label 5150 3200 0    50   ~ 0
 LED_SIGNAL_RED
-Text Label 5150 1550 0    50   ~ 0
+Text Label 7350 3200 2    50   ~ 0
 LED_SIGNAL_ORANGE
-Text Label 7550 1450 2    50   ~ 0
+Text Label 7550 3100 2    50   ~ 0
 LED_SIGNAL_GREEN
-Text Label 7550 1550 2    50   ~ 0
+Text Label 4950 3300 0    50   ~ 0
 LED_SIGNAL_GREEN2
 Wire Wire Line
-	6500 1450 7550 1450
-Wire Wire Line
-	6500 1550 7550 1550
-Wire Wire Line
-	5150 1450 6000 1450
-Wire Wire Line
-	5150 1550 6000 1550
+	6500 3100 7550 3100
+Wire Wire Line
+	6000 3300 4950 3300
+Wire Wire Line
+	5150 3200 6000 3200
+Wire Wire Line
+	7350 3200 6500 3200
 Text Label 7900 1350 0    50   ~ 0
 LED_SIGNAL_GREEN
@@
 Wire Wire Line
 	7850 5050 7850 5400
+NoConn ~ 6500 1450
+NoConn ~ 6500 1550
+NoConn ~ 6000 1550
+NoConn ~ 6000 1450
 Wire Bus Line
 	9100 4150 9100 4350

Commit message: シルクで1ピンマーク追記
Connections:
- net ThermistorIn: now reaches J11.18 (Pin_18)
- no-connect marks 47 -> 46
Changed lines of the file:
@@
 $Descr A4 11693 8268
 encoding utf-8
-Sheet 3 9
+Sheet 3 10
 Title ""
 Date ""
@@
 	3200 2250 3800 2250
 NoConn ~ 2700 2150
-NoConn ~ 3200 2150
 $Comp
 L Device:C C?
@@
 NoConn ~ 6000 1550
 NoConn ~ 6000 1450
+Text HLabel 3800 2150 2    50   Input ~ 0
+ThermistorIn
+Wire Wire Line
+	3800 2150 3200 2150
 Wire Bus Line
 	9100 4150 9100 4350
