File: HW/file5FF7CDA9.sch (KiCad schematic (older format))
At the start: 15 parts, among them K1 G5Q-14_DC5, K2 G5Q-14_DC5, K3 G5Q-14_DC5, Q1 2SC1815, Q2 2SC1815, Q3 2SC1815

Commit message: Ethernetボードの配置のためにレイアウト変更
Connections:
- net FAN_DRIVE_HOT: now also K2.3; no longer K2.4
- net HEATER_DRIVE_HOT: now also K3.3; no longer K3.4
- net UV_DRIVE_HOT: now also K1.3; no longer K1.4
Changed lines of the file:
@@
 	7300 2350 7150 2350
 Connection ~ 7300 2350
-NoConn ~ 4100 1250
-NoConn ~ 8250 1300
-NoConn ~ 4100 4000
 Wire Wire Line
 	4250 4600 4000 4600
@@
 	4250 1850 4000 1850
 Wire Wire Line
-	3900 950  3900 1250
+	4100 950  4100 1250
 Connection ~ 3600 5250
 Wire Wire Line
@@
 	1    0    0    -1
 $EndComp
-Text HLabel 3750 950  0    50   Output ~ 0
+Text HLabel 3950 950  0    50   Output ~ 0
 UV_DRIVE_HOT
-Text HLabel 7950 850  0    50   Output ~ 0
+Text HLabel 8150 850  0    50   Output ~ 0
 HEATER_DRIVE_HOT
-Text HLabel 3650 3750 0    50   Output ~ 0
+Text HLabel 3850 3750 0    50   Output ~ 0
 FAN_DRIVE_HOT
 Wire Wire Line
-	8050 850  7950 850
+	8250 850  8150 850
 Wire Wire Line
-	8050 850  8050 1300
+	8250 850  8250 1300
 Wire Wire Line
-	3900 950  3750 950
+	4100 950  3950 950
 Text HLabel 4900 3850 0    50   Input ~ 0
 AC100V_COLD
@@
 	4900 3850 5300 3850
 Wire Wire Line
-	3900 3750 3650 3750
+	4100 3750 3850 3750
 Wire Wire Line
-	3900 3750 3900 4000
+	4100 3750 4100 4000
 Text HLabel 4250 4600 2    50   Input ~ 0
 AC100V_HOT
@@
 Wire Wire Line
 	3600 4000 3600 3850
+NoConn ~ 3900 1250
+NoConn ~ 8050 1300
+NoConn ~ 3900 4000
 Wire Bus Line
 	9650 3600 9650 4200
